File: Sensor_Board_Try2.brd (EAGLE design)
At the start: 69.8 x 64.4 mm, 28 parts, among them IC1 AT24CP, IC3 DS1307, Q1 BSS123, Q2 BSS123, Q3 32.768

Commit message: Add files via upload
Parts:
- added R10: 4.7K, adafruit:M1406
- moved J4 63.1 mm to (68.1, 23.4), turned to 180 degrees
- moved J2 59.6 mm to (68.1, 16.8), turned to 180 degrees
- moved J5 58.2 mm to (68.1, 29.7), turned to 180 degrees
- moved R7 58.2 mm to (72.1, 29.5), turned to 90 degrees
- moved R8 56.4 mm to (72.1, 36.3), turned to 90 degrees
- moved R6 53.2 mm to (72.1, 21.8), turned to 90 degrees
- moved R12 49.0 mm to (31.8, 53.3)
- moved R11 45.5 mm to (31.8, 58.4), turned to 180 degrees
- moved JP2 34.6 mm to (14.5, 58.4), turned to 180 degrees
- moved IC3 32.9 mm to (48.3, 8.38)
- moved Q3 29.2 mm to (38.9, 4.57), turned to 90 degrees
- moved JP3 27.3 mm to (14.5, 54.9), turned to 180 degrees
- moved SV3 26.6 mm to (52.3, 55.9), turned to 0 degrees
- moved C1 24.1 mm to (52.8, 44.5), turned to 270 degrees
- moved J3 24.0 mm to (14.0, 22.9), turned to 0 degrees
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Connections:
- net 5V: now also R10.1
- net SQW: now also R10.2
Routing:
- net SDA: track 105.2 -> 173.6 mm
- net PD7: track 74.9 -> 19.6 mm
- net 5V: track 214.6 -> 162.2 mm
- net PD6: track 66.0 -> 18.0 mm
- net PD5: track 55.4 -> 16.9 mm
- net SCL: track 100.7 -> 138.8 mm, vias 1 -> 0
- net SDAL: track 74.4 -> 38.4 mm
- net 3V: track 201.3 -> 182.5 mm
- net RESET: track 36.7 -> 18.5 mm
- net A2: track 4.86 -> 22.3 mm
- net SCLL: track 34.4 -> 50.4 mm
- net A1: track 5.08 -> 15.1 mm
- net N$14: track 17.8 -> 11.0 mm
- net SQW: track 0.00 -> 5.75 mm
- net N$15: track 15.2 -> 10.6 mm
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