File: Sensor_Board_Try2.brd (EAGLE design)
At the start: 69.8 x 64.4 mm, 32 parts, among them IC1 AT24CP, IC3 DS1307, Q1 BSS123, Q2 BSS123, Q3 32.768

Commit message: final version of the boards
Connections:
- net N$6 renamed VBAT
Changed lines of the file:
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@@
 <wire x1="13.208" y1="40.64" x2="14.478" y2="41.91" width="0.4064" layer="1"/>
 </signal>
-<signal name="N$6">
+<signal name="VBAT">
 <contactref element="IC3" pad="3"/>
 <contactref element="G1" pad="+@1"/>
