File: eagle/Sensor_Board_Try2.sch (EAGLE design)
At the start: 28 parts, among them IC1 AT24CP, IC3 DS1307, Q1 BSS123, Q2 BSS123, Q3 32.768

Commit message: moved the boards into eagle folder
Parts:
- removed R12: 4.7K, adafruit:R-US_M1406
- removed R4: 10K, resistor:R-US_M1406
- removed R5: 10k, rcl:R-US_M1406
- removed R8: 4.7K, resistor:R-US_M1406
- added C2, C3: 12.5pF, eagle-ltspice:C
- added C4, C5: (no value), rcl:CPOL-USE2-4
- added G1: 10MM_SM_COIN_CELL_CLIP, battery:10MM_SM_COIN_CELL_CLIP
- added R13: 10k, rcl:R-US_M0805
- added R14, R9: 4.7k, rcl:R-US_M0805
- JP2: value JUMPER-SMT_3_1-NC_TRACE_SILK -> JP2
- JP3: value JUMPER-SMT_3_1-NC_TRACE_SILK -> JP3
- JP4: value JUMPER-SMT_3_1-NC_TRACE_SILK -> JP4
- R1, R2, R3: value 10K -> 10k; device resistor:R-US_M1406 -> rcl:R-US_M0805
- R11: value 4.7K -> 10k; device adafruit:R-US_M1406 -> rcl:R-US_M0805
- R6, R7: value 4.7K -> 4.7k; device resistor:R-US_M1406 -> rcl:R-US_M0805
Connections:
- removed net N$6: IC3.VBAT
- new net VBAT: G1.+, IC3.VBAT
- net 3V: now also C5.+, R11.2, R2.2; no longer R1.2, R3.2
- net 5V: now also C4.+, R1.2, R13.2, R14.2, R3.2, R9.2; no longer R11.1, R12.2, R2.2, R4.2, R5.1, R8.2
- net GND: now also C2.2, C3.2, C4.-, C5.-, G1.-
- net N$14: now also C2.1
- net N$15: now also C3.1
- net PD5: now also R9.1; no longer R6.1
- net PD6: now also R6.1; no longer R7.1
- net PD7: now also R7.1; no longer R8.1
- net RESET: now also R13.1; no longer R5.2
- net SCL: now also R3.1; no longer R11.2, R4.1
- net SCLL: now also R2.1; no longer R3.1
- net SDA: now also R1.1; no longer R12.1, R2.1
- net SDAL: now also R11.1; no longer R1.1
- net SQW: now also R14.1
Other:
- moved on the sheet: Q3, R1, R11, R2, R3, R6, R7
